File: hardware/nrfmicro.kicad_sch (KiCad schematic)
At the start: 24 parts, among them J1 USB-C USB 2.0 MC-372, J2 Conn_01x04, J3 Conn_01x02, J4 Conn_01x04, Q1 AO3407, Q2 AO3407, U1 E73-2G4M08S1C, U2 AP2112K-3.3, U3 TP4054, U4 ProMicro, X1 32768kHz

Commit message: v0.1
Parts:
- D2: value BLUE -> WHITE; LCSC (none) -> C2290
- D3: LCSC (none) -> C2286
- J1: footprint nrfmicro:USB-C_C168688 -> custom:GT-USB-7047B; symbol nrfmicro:USB_C_Receptacle_USB2.0 -> Connector:USB_C_Receptacle_USB2.0; LCSC (none) -> C963217
- J2, J4, U4: now left out of the parts list
- J3: footprint (none) -> nrfmicro:connector_bat; now left out of the parts list
- Q1, Q2, U3: JLCPCB Rotation Offset (none) -> 180
- R1, R2, R3, R4, R6, R7, R8, R9: footprint Resistor_SMD:R_0603_1608Metric -> Resistor_SMD:R_0402_1005Metric
- R5: value RPROG -> 10K; footprint Resistor_SMD:R_0603_1608Metric -> Resistor_SMD:R_0402_1005Metric
- U2: value AP2112K-3.3 -> XC6220B331MR; LCSC (none) -> C86534
- X1: footprint (none) -> custom:Q13FC1350000400; LCSC (none) -> C32346
Connections:
- net GND: now also J1.A12 (GND), J1.B1 (GND), J1.B12 (GND)
- net VBUS: now also J1.A9 (VBUS), J1.B4 (VBUS), J1.B9 (VBUS)
- net BLUE_LED renamed WHITE_LED
